File: MJoy16-C1.sch (EAGLE design)
At the start: 31 parts, among them J1 PN61729-S, Q1 12MHz, U1 MEGA16-P

Commit message: Added board and Eagle3D files
Parts:
- C4, C5, C6: device rcl:C-US025-024X044 -> rcl:C-US050-025X075
- D1, D2: device diode:BZX90 -> diode:ZENER-DIODEZD-5
- renumbered Q1 to X1
